File: esp8266_board.sch (KiCad schematic (older format))
At the start: 11 parts, among them P1 CONN_01X11, P2 CONN_01X11, U1 ESP-12F, U2 AP111733

Commit message: v1
Parts:
- removed U2: AP111733, TO_SOT_Packages_SMD:SOT-223, symbol AP111733
- added U2: AMS1117-3V3, TO_SOT_Packages_SMD:SOT-223, symbol AMS1117-3V3
- C1, C2, C3: footprint Capacitor_SMD:C_0805_2012Metric -> Capacitors_SMD:C_0805_HandSoldering
- P1, P2: footprint Connector_PinHeader_2.54mm:PinHeader_1x11_P2.54mm_Vertical -> Pin_Headers:Pin_Header_Straight_1x11
- R1, R2: value 2k -> 10k; footprint Resistor_SMD:R_0805_2012Metric -> Resistors_SMD:R_0805_HandSoldering
- R3: value 1k -> 2k; footprint Resistor_SMD:R_0805_2012Metric -> Resistors_SMD:R_0805_HandSoldering
- R4: footprint Resistor_SMD:R_0805_2012Metric -> Resistors_SMD:R_0805_HandSoldering
Connections:
- net +5V: now also U2.3 (VI)
- net GND: now also R3.1, U2.1 (GND/ADJ); no longer R1.1, R2.1
- net at R1.2, U1.1 (REST): now also P1.1 (P1); no longer R3.1
- net at U1.15 (RXD): now also R3.2, R4.2; no longer P2.2 (P2)
- net at R2.2, U1.3 (CH_PD): now also P1.3 (P3); no longer R4.1
- net +3V3: now reaches C2.1, C3.1, U1.8 (VCC)
- net +3V3: now also R1.1, R2.1, U2.2 (VO), U2.4 (PAD)
- new net: P2.2 (P2), R4.1
